File: hw/xdeya.kicad_pcb (KiCad board)
At the start: 2 copper layers, 91.2 x 50 mm, 71 parts, among them J10 A, J11 A, J12 A, J2 display, J3 antenna, J4 USB_B_Micro, J5 battery, J6 A, J7 K, J9 A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

Commit message: hw - тестовый вариант с антенным усилителем
Parts:
- removed J10, J11, J12, J9: A, MHole:SolderWirePad_1x01_SMD_3x6mm
- removed R14: 10, Resistor_SMD:R_0805_2012Metric
- added C16: 470pF, Capacitor_SMD:C_0805_2012Metric, F.Cu at (65.0, 46.7)
- added C17: 1μF, Capacitor_SMD:C_0805_2012Metric, F.Cu at (71.2, 52.5)
- added J1: ant, rfshield:BMI_16.5x16mm, F.Cu at (66.3, 52.0)
- added U8: 2659, maxdfn:DFN150X100X80-6N, F.Cu at (71.2, 48.8)
- L1: value 27nH -> 6,8nH
- moved L1 26.0 mm to (66.0, 49.3), turned to 0 degrees
- moved J3 21.3 mm to (65.0, 40.7)
- moved U6 8.20 mm to (84.0, 51.0)
- moved H1 4.86 mm to (53.3, 83.3)
- moved H2 4.86 mm to (53.3, 40.4)
- moved H4 0.06 mm to (132.5, 83.3)
Connections:
- J3 pad 1: Net-(J3-Pad1) -> Net-(C16-Pad2)
- L1 pad 2: Net-(J3-Pad1) -> Net-(L1-Pad2)
- U6 pad 11: Net-(J3-Pad1) -> Net-(U6-Pad11)
Routing:
- net Net-(U6-Pad14): track 0.00 -> 13.4 mm, vias 0 -> 2
- net Net-(C17-Pad1): track 3.78 -> 16.6 mm
- net Net-(U6-Pad11): track 0.00 -> 9.17 mm
- net /gps-rx: track 27.3 -> 36.2 mm
- net /gps-tx: track 27.6 -> 36.2 mm
- net Net-(J3-Pad1): track 8.61 -> 0.00 mm
- net hwpwr: track 10.5 -> 18.0 mm
- net Net-(L1-Pad2): track 0.00 -> 3.62 mm
- net Net-(C16-Pad2): track 0.00 -> 3.58 mm
- net GND: track 22.3 -> 24.6 mm, vias 52 -> 182
- net +3V3: track 208.7 -> 207.6 mm
- net Net-(C16-Pad1): track 2.23 -> 1.60 mm
Other:
- board size 91.2 x 50 mm -> 86.2 x 50 mm
- board text added: "XDE-YA v0.4.2 test"
- board text removed: "Antenna"
- board text removed: "GPS-adv v0.4.1"
