File: hw/xdeya.kicad_pcb (KiCad board)
At the start: 2 copper layers, 86.2 x 48.5 mm, 70 parts, among them J2 display, J3 antenna, J4 USB_B_Micro, J5 battery, J6 A, J7 K, Q5 UMH3N, SW3 btn-up, SW4 btn-sel, SW5 btn-down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

Commit message: hw - небольшие доработки
Parts:
- moved R18 3.18 mm to (121.9, 74.2)
- moved R19 1.23 mm to (124.1, 74.2)
Connections:
- R18 pad 2: /s-tx -> /s-rx
- R19 pad 2: /s-rx -> /s-tx
Routing:
- net Net-(U7-TXD): track 6.90 -> 2.16 mm
- net Net-(Q5A-E1): track 9.68 -> 12.3 mm
- net Net-(U7-RXD): track 2.32 -> 3.13 mm
- net /s-tx: track 2.98 -> 2.17 mm
- net /s-rx: track 2.20 -> 2.77 mm
- net GND: vias 155 -> 163
Other:
- board text added: "XDE-YA v0.6-t2"
- board text removed: "XDE-YA v0.6-t1"
