File: hw/xdeya.kicad_sch (KiCad schematic)
At the start: 75 parts, among them J2 display, J3 antenna, J4 USB_B_Micro, J5 battery, J6 A, J7 K, Q1 ML5203, Q2 ML5203, Q3 S8050, Q4 S8050, SW3 btn-up, SW4 btn-sel, SW5 btn-down, U1 ESP32-WROOM-32, U2 MCP73831, U3 MIC5219-3.3, U4 BMP280, U5 PCF8563T, U6 NEO-M8N, U7 CP2102, U8 LSM303DLH, U9 XC6206P182MR, Y1 32768

Commit message: hw - схема с использованием axp2101
Parts:
- removed C14: 1μF, Capacitor_SMD:C_0805_2012Metric, symbol Device:C
- removed C18: 4,7μF, Capacitor_SMD:C_0805_2012Metric, symbol Device:C
- removed Q1, Q2: ML5203, Package_TO_SOT_SMD:SOT-23, symbol Device:Q_PMOS_GSD
- removed Q3, Q4: S8050, Package_TO_SOT_SMD:SOT-23, symbol Device:Q_NPN_BEC
- removed R1, R12: 100k, Resistor_SMD:R_0805_2012Metric, symbol Device:R
- removed R13, R5: 510, Resistor_SMD:R_0805_2012Metric, symbol Device:R
- removed R6, R7, R8: 150k, Resistor_SMD:R_0805_2012Metric, symbol Device:R
- removed U2: MCP73831, Package_TO_SOT_SMD:SOT-23-5, symbol Battery_Management:MCP73831-2-OT
- removed U3: MIC5219-3.3, Package_TO_SOT_SMD:SOT-23-5, symbol Regulator_Linear:MIC5219-3.3YM5
- removed U8: LSM303DLH, lsm303dlh:LGA28R55P7X7_500X500X100, symbol lsm303dlh:LSM303DLH
- removed U9: XC6206P182MR, Package_TO_SOT_SMD:SOT-23, symbol Regulator_Linear:XC6206PxxxMR
- added C11, C20, C21, C23: 10μF, Capacitor_SMD:C_0805_2012Metric, symbol Device:C
- added C22: 22μF, Capacitor_SMD:C_0805_2012Metric, symbol Device:C
- added C24, C25, C26: 1μF, Capacitor_SMD:C_0805_2012Metric, symbol Device:C
- added C27: 4,7μF, Capacitor_SMD:C_0805_2012Metric, symbol Device:C
- added D2: 1N5819, Diode_SMD:D_SOD-323, symbol Device:D
- added L2: 2.2μH/1.5A, Inductor_SMD_Wurth:L_Wurth_WE-LQSH-3012, symbol Device:L
- added Q5: UMH3N, Package_TO_SOT_SMD:SOT-363_SC-70-6, symbol Transistor_BJT:UMH3N
- added R24: 47k, Resistor_SMD:R_0805_2012Metric, symbol Device:R
- added U10: AXP2101, Package_DFN_QFN:QFN-40-1EP_5x5mm_P0.4mm_EP3.6x3.6mm, symbol axp2101:axp2101
- added U2: LSM303AGR, PQFN50P200X200X100-12N, symbol lsm303agr:LSM303AGR
- C3: value 4,7μF -> 10μF
- C6: value 470p -> 1μF
- C7: value 1μF -> 4,7μF
- L1: symbol Device:L_Ferrite -> Device:L
- R11: value 4k7 -> 100
- R16, R17: value 10k -> 1
Connections:
- net +3.3V: now also C22.1, L2.2, U10.21 (FB1); no longer C13.1, C16.1, C4.1, R3.2, U1.3 (EN), U4.6 (VDDIO), U4.8 (VDD), U5.8 (VDD), U6.22 (V_BCKP), XS1.4 (Vdd)
- net GND: now also C17.2, R11.1, C11.2, C20.1, C21.2, C22.2, C23.2, C24.2, C25.2, C26.2, C27.2, U10.3 (GND), U10.41 (GND), U2.6 (GND), U2.8 (GND); no longer R11.2
- net i2c-scl: now also U10.40 (SCK)
- net i2c-sda: now also U10.39 (SDA)
- net s-boot: now also Q5.3 (C2)
- net DLIGHT: now reaches R15.2
- net DLIGHT: now also U10.19 (ALDO2)
- net VNAVI: now reaches C6.1
- net VNAVI: now also U6.23 (VCC), U10.16 (ALDO3)
- net at U7.11 (~{SUSPEND}): no longer R21.1
- net at U7.12 (SUSPEND): now also R21.1
- net at U7.23 (~{CTS}): no longer R19.1
- net at U7.24 (~{RTS}): now also Q5.1 (E1), Q5.5 (B2); no longer R18.1
- net at U7.25 (RXD): now also R19.1; no longer R16.2
- net at U7.26 (TXD): now also R18.1
- net at U7.28 (~{DTR}): now also Q5.2 (B1), Q5.4 (E2); no longer R17.1
- net at U7.4 (D+): now also J4.3 (D+)
- net at U7.9 (~{RST}): now also R20.1
- net at R16.1: now also C21.1, U10.17 (ALDOIN)
- net VSYS: now reaches R17.2
- net VSYS: now also R16.2, C20.2, U10.23 (VIN1), U10.34 (VSYS), U10.36 (VMID)
- net VBUS: now reaches R20.2
- net VBUS: now also C2.1, J4.1 (VBUS), U7.7 (VREGIN), U7.8 (VBUS), C11.1, U10.37 (VBUS)
- net at C17.1: now also U2.5 (C1)
- net at R23.2: now also U2.4 (SDA/SDI/SDO)
- net at R22.1: now also U2.1 (SCL/SPC)
- net +1V8 renamed VCOMP-IO
- net VCOMP-IO: now also U10.12 (BLDO1), U2.10 (VDD_IO), U2.2 (CS_XL), U2.3 (CS_MAG)
- net +BATT: no longer names the net of C3.1, J5.1 (Pin_1)
- net +BATT: now also U10.33 (BAT)
- net b-sel renamed PWROK
- net PWROK: now also U10.29 (PWROK)
- net batt-chk renamed CHRGIRQ
- net CHRGIRQ: now also R24.1, U10.38 (IRQ)
- net chg-ind: no longer names the net of U1.14 (IO12)
- net d-led: no longer names the net of U1.8 (IO32)
- net hwen: no longer names the net of U1.12 (IO27)
- net hwpwr renamed VCOMP-SUPP
- net VCOMP-SUPP: now also U10.14 (BLDO2), U2.9 (VDD); no longer U6.23 (VCC)
- removed net usb-5v: C2.1, J4.1 (VBUS), R20.1, U7.7 (VREGIN)
- removed net usb-d+: J4.3 (D+), U7.8 (VBUS)
- net usb-d-: no longer names the net of J4.2 (D-), U7.5 (D-)
- new net: C25.1, U10.10 (CPULDOS)
- new net: C23.1, R17.1, U10.13 (BLDOIN)
- new net: C24.1, U10.2 (VREF)
- new net: L2.1, U10.22 (LX1)
- new net: R11.2, U10.31 (TS)
- new net PWRON: D2.1 (K), U10.30 (PWRON)
- new net VBMP: C27.1, U10.18 (ALDO1), U4.6 (VDDIO), U4.8 (VDD)
- new net VRTC: C26.1, C4.1, R24.2, U10.28 (VRTC), U5.8 (VDD), U6.22 (V_BCKP)
- new net VSDCARD: C16.1, U10.15 (ALDO4), XS1.4 (Vdd)
- new net s-en: C13.1, D2.2 (A), Q5.6 (C1), R3.2, U1.3 (EN)
Other:
- moved on the sheet: C10, C12, C13, C16, C17, C19, C2, C3, C5, C8, C9, D1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

Commit message: hw - примерная расстановка элементов
Parts:
- removed C12: 1μF, Capacitor_SMD:C_0805_2012Metric, symbol Device:C
- removed D1: 1N5819, Diode_SMD:D_SOD-323, symbol Device:D
- U2: footprint PQFN50P200X200X100-12N -> lsm303agr:PQFN50P200X200X100-12N
- Y1: footprint Crystal:Crystal_AT310_D3.0mm_L10.0mm_Vertical -> Crystal:Crystal_DS26_D2.0mm_L6.0mm_Horizontal_1EP_style2; symbol Device:Crystal -> Device:Crystal_GND3
Connections:
- net GND: now also Y1.3
- net VBUS: now also R20.1; no longer R20.2
- net at U7.9 (~{RST}): now also R20.2; no longer R20.1
Other:
- moved on the sheet: R20
Changed lines of the file:
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@@
   (junction (at 184.15 109.22) (diameter 0) (color 0 0 0 0)
   )
+  (junction (at 177.8 33.02) (diameter 0) (color 0 0 0 0)
+  )
   (junction (at 54.61 132.08) (diameter 0) (color 0 0 0 0)
   )
@@
   (junction (at 157.48 15.24) (diameter 0) (color 0 0 0 0)
   )
-  (junction (at 246.38 40.64) (diameter 0) (color 0 0 0 0)
-  )
   (junction (at 36.83 54.61) (diameter 0) (color 0 0 0 0)
   )
@@
     (stroke (width 0) (type default))
   )
-  (wire (pts (xy 240.03 40.64) (xy 240.03 49.53))
-    (stroke (width 0) (type default))
-  )
   (wire (pts (xy 34.29 129.54) (xy 44.45 129.54))
     (stroke (width 0) (type default))
@@
     (stroke (width 0) (type default))
   )
-  (wire (pts (xy 257.81 40.64) (xy 259.08 40.64))
-    (stroke (width 0) (type default))
-  )
   (wire (pts (xy 237.49 49.53) (xy 237.49 48.26))
     (stroke (width 0) (type default))
@@
     (stroke (width 0) (type default))
   )
+  (wire (pts (xy 184.15 33.02) (xy 177.8 33.02))
+    (stroke (width 0) (type default))
+  )
   (wire (pts (xy 137.16 105.41) (xy 137.16 110.49))
     (stroke (width 0) (type default))
   )
-  (wire (pts (xy 177.8 34.29) (xy 177.8 31.75))
+  (wire (pts (xy 177.8 34.29) (xy 177.8 33.02))
     (stroke (width 0) (type default))
   )
@@
     (stroke (width 0) (type default))
   )
-  (wire (pts (xy 246.38 40.64) (xy 240.03 40.64))
-    (stroke (width 0) (type default))
-  )
   (bus (pts (xy 105.41 80.01) (xy 105.41 81.28))
     (stroke (width 0) (type default))
@@
     (stroke (width 0) (type default))
   )
+  (wire (pts (xy 177.8 33.02) (xy 177.8 31.75))
+    (stroke (width 0) (type default))
+  )
   (wire (pts (xy 336.55 123.19) (xy 336.55 124.46))
     (stroke (width 0) (type default))
@@
     (stroke (width 0) (type default))
   )
+  (wire (pts (xy 184.15 27.94) (xy 184.15 33.02))
+    (stroke (width 0) (type default))
+  )
   (wire (pts (xy 179.07 53.34) (xy 182.88 53.34))
     (stroke (width 0) (type default))
@@
     (stroke (width 0) (type default))
   )
-  (wire (pts (xy 250.19 40.64) (xy 246.38 40.64))
-    (stroke (width 0) (type default))
-  )
   (wire (pts (xy 80.01 67.31) (xy 90.17 67.31))
     (stroke (width 0) (type default))
@@
     )
   )
-  (symbol (lib_id "Device:Crystal") (at 189.23 27.94 270) (unit 1)
+  (symbol (lib_id "Device:Crystal_GND3") (at 189.23 27.94 270) (unit 1)
     (in_bom yes) (on_board yes) (dnp no)
     (property "Reference" "Y1" (at 192.5574 26.7716 90)
@@
       (effects (font (size 1.27 1.27)) (justify left))
     )
-    (property "Footprint" "Crystal:Crystal_AT310_D3.0mm_L10.0mm_Vertical" (at 189.23 27.94 0)
+    (property "Footprint" "Crystal:Crystal_DS26_D2.0mm_L6.0mm_Horizontal_1EP_style2" (at 189.23 27.94 0)
       (effects (font (size 1.27 1.27)) hide)
     )
@@
     (pin "1")
     (pin "2")
+    (pin "3")
     (instances
       (project "xdeya"
@@
   (symbol (lib_id "Device:C") (at 177.8 27.94 0) (unit 1)
     (in_bom yes) (on_board yes) (dnp no)
-    (property "Reference" "C5" (at 180.721 26.7716 0)
+    (property "Reference" "C5" (at 171.45 26.8986 0)
       (effects (font (size 1.27 1.27)) (justify left))
     )
-    (property "Value" "22pF" (at 180.721 29.083 0)
+    (property "Value" "22pF" (at 171.45 29.21 0)
       (effects (font (size 1.27 1.27)) (justify left))
     )
@@
     )
   )
-  (symbol (lib_id "Device:R") (at 222.25 54.61 270) (unit 1)
+  (symbol (lib_id "Device:R") (at 222.25 54.61 90) (unit 1)
     (in_bom yes) (on_board yes) (dnp no)
-    (property "Reference" "R20" (at 220.98 57.15 90)
+    (property "Reference" "R20" (at 223.52 52.07 90)
       (effects (font (size 1.27 1.27)) (justify left))
     )
-    (property "Value" "10k" (at 220.98 59.69 90)
+    (property "Value" "10k" (at 223.52 49.53 90)
       (effects (font (size 1.27 1.27)) (justify left))
     )
-    (property "Footprint" "Resistor_SMD:R_0805_2012Metric" (at 222.25 52.832 90)
+    (property "Footprint" "Resistor_SMD:R_0805_2012Metric" (at 222.25 56.388 90)
       (effects (font (size 1.27 1.27)) hide)
     )
@@
     )
   )
-  (symbol (lib_id "power:+3.3V") (at 259.08 40.64 270) (unit 1)
-    (in_bom yes) (on_board yes) (dnp no)
-    (property "Reference" "#PWR04" (at 255.27 40.64 0)
-      (effects (font (size 1.27 1.27)) hide)
-    )
-    (property "Value" "+3.3V" (at 262.3312 41.021 90)
-      (effects (font (size 1.27 1.27)) (justify left))
-    )
-    (property "Footprint" "" (at 259.08 40.64 0)
-      (effects (font (size 1.27 1.27)) hide)
-    )
-    (property "Datasheet" "" (at 259.08 40.64 0)
-      (effects (font (size 1.27 1.27)) hide)
-    )
-    (pin "1")
-    (instances
-      (project "xdeya"
-        (path "/81c4e96a-f93b-443f-91d4-080d23f47ded"
-          (reference "#PWR04") (unit 1)
-        )
-      )
-    )
-  )
-  (symbol (lib_id "Device:C") (at 246.38 44.45 180) (unit 1)
-    (in_bom yes) (on_board yes) (dnp no)
-    (property "Reference" "C12" (at 252.73 43.18 0)
-      (effects (font (size 1.27 1.27)) (justify left))
-    )
-    (property "Value" "1μF" (at 252.73 45.72 0)
-      (effects (font (size 1.27 1.27)) (justify left))
-    )
-    (property "Footprint" "Capacitor_SMD:C_0805_2012Metric" (at 245.4148 40.64 0)
-      (effects (font (size 1.27 1.27)) hide)
-    )
-    (property "Datasheet" "~" (at 246.38 44.45 0)
-      (effects (font (size 1.27 1.27)) hide)
-    )
-    (pin "1")
-    (pin "2")
-    (instances
-      (project "xdeya"
-        (path "/81c4e96a-f93b-443f-91d4-080d23f47ded"
-          (reference "C12") (unit 1)
-        )
-      )
-    )
-  )
-  (symbol (lib_id "power:GND") (at 246.38 48.26 0) (unit 1)
-    (in_bom yes) (on_board yes) (dnp no)
-    (property "Reference" "#PWR0125" (at 246.38 54.61 0)
-      (effects (font (size 1.27 1.27)) hide)
-    )
-    (property "Value" "GND" (at 250.19 49.53 0)
-      (effects (font (size 1.27 1.27)))
-    )
-    (property "Footprint" "" (at 246.38 48.26 0)
-      (effects (font (size 1.27 1.27)) hide)
-    )
-    (property "Datasheet" "" (at 246.38 48.26 0)
-      (effects (font (size 1.27 1.27)) hide)
-    )
-    (pin "1")
-    (instances
-      (project "xdeya"
-        (path "/81c4e96a-f93b-443f-91d4-080d23f47ded"
-          (reference "#PWR0125") (unit 1)
-        )
-      )
-    )
-  )
-  (symbol (lib_id "Device:D") (at 254 40.64 180) (unit 1)
-    (in_bom yes) (on_board yes) (dnp no)
-    (property "Reference" "D1" (at 254 35.1282 0)
-      (effects (font (size 1.27 1.27)))
-    )
-    (property "Value" "1N5819" (at 254 37.4396 0)
-      (effects (font (size 1.27 1.27)))
-    )
-    (property "Footprint" "Diode_SMD:D_SOD-323" (at 254 40.64 0)
-      (effects (font (size 1.27 1.27)) hide)
-    )
-    (property "Datasheet" "~" (at 254 40.64 0)
-      (effects (font (size 1.27 1.27)) hide)
-    )
-    (pin "1")
-    (pin "2")
-    (instances
-      (project "xdeya"
-        (path "/81c4e96a-f93b-443f-91d4-080d23f47ded"
-          (reference "D1") (unit 1)
-        )
-      )
-    )
-  )
   (symbol (lib_id "Device:L") (at 24.13 143.51 0) (unit 1)
     (in_bom yes) (on_board yes) (dnp no)
@@
       (effects (font (size 1.27 1.27)))
     )
-    (property "Footprint" "PQFN50P200X200X100-12N" (at 115.57 170.18 0)
+    (property "Footprint" "lsm303agr:PQFN50P200X200X100-12N" (at 115.57 170.18 0)
       (effects (font (size 1.27 1.27)) (justify bottom) hide)
     )

Commit message: hw - доделана трассировка платы, но скорее всего, придётся всё переделывать, слишком много пересечений
Parts:
- U10: footprint Package_DFN_QFN:QFN-40-1EP_5x5mm_P0.4mm_EP3.6x3.6mm -> Package_DFN_QFN:QFN-40-1EP_5x5mm_P0.4mm_EP3.6x3.6mm_ThermalVias
Connections:
- net batt: now reaches C3.1, J5.1 (Pin_1), U10.33 (BAT)
Changed lines of the file:
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@@
     (effects (font (size 1.27 1.27)) (justify right bottom))
+  )
+  (label "batt" (at 349.25 34.29 0) (fields_autoplaced)
+    (effects (font (size 1.27 1.27)) (justify left bottom))
   )
   (label "spi-miso" (at 81.28 69.85 0) (fields_autoplaced)
@@
       (effects (font (size 1.27 1.27)) (justify left))
     )
-    (property "Footprint" "Package_DFN_QFN:QFN-40-1EP_5x5mm_P0.4mm_EP3.6x3.6mm" (at 378.46 129.54 0)
+    (property "Footprint" "Package_DFN_QFN:QFN-40-1EP_5x5mm_P0.4mm_EP3.6x3.6mm_ThermalVias" (at 378.46 129.54 0)
       (effects (font (size 1.27 1.27) italic) hide)
     )

Commit message: hw - переделана трассировка платы, стало лучше, осталось: расставить шелкографию, проверить, наделать переходных по gnd
Parts:
- removed C1: 10μF, Capacitor_SMD:C_0805_2012Metric, symbol Device:C
Connections:
- net CHRGIRQ: now also R24.2; no longer R24.1
- net GND: now also C11.1, C13.1, C21.1, C23.1, C5.1, R11.2; no longer C11.2, C13.2, C21.2, C23.2, C5.2, R11.1
- net VBUS: now also C11.2; no longer C11.1
- net VRTC: now also R24.1; no longer R24.2
- net VSYS: now also R16.1, R17.1; no longer R16.2, R17.2
- net s-en: now also C13.2; no longer C13.1
- net at Y1.2: now also C5.2, U5.1 (OSCI); no longer U5.2 (OSCO)
- net at U10.31 (TS): now also R11.1; no longer R11.2
- new net: U5.2 (OSCO), Y1.1
- new net: C23.2, R17.2, U10.13 (BLDOIN)
- new net: C21.2, R16.2, U10.17 (ALDOIN)
Other:
- moved on the sheet: C11, C13, C21, C23, C5, R11, R16, R17, R24
