File: hw/xdeya.kicad_sch (KiCad schematic)
At the start: 70 parts, among them J2 display, J3 antenna, J4 USB_B_Micro, J5 battery, J6 A, J7 K, Q5 UMH3N, SW3 btn-up, SW4 btn-sel, SW5 btn-down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

Commit message: hw - небольшие доработки
Connections:
- net s-rx: now also R18.2; no longer R19.2
- net s-tx: now also R19.2; no longer R18.2
Changed lines of the file:
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@@
     (effects (font (size 1.27 1.27)) (justify right bottom))
   )
-  (label "s-rx" (at 274.32 22.86 0) (fields_autoplaced)
+  (label "s-rx" (at 274.32 20.32 0) (fields_autoplaced)
     (effects (font (size 1.27 1.27)) (justify left bottom))
   )
@@
     (effects (font (size 1.27 1.27)) (justify left bottom))
   )
-  (label "s-tx" (at 274.32 20.32 0) (fields_autoplaced)
+  (label "s-tx" (at 274.32 22.86 0) (fields_autoplaced)
     (effects (font (size 1.27 1.27)) (justify left bottom))
   )
